File: Loren_Hackpad/PCB/LorenHackpad.kicad_pcb (KiCad board)
At the start: 2 copper layers, 80.8 x 90.6 mm, 27 parts, among them J1 OLED_display, SW1 SW_Push, SW10 SW_Push, SW2 RotaryEncoder_Switch, SW3 SW_Push, SW4 SW_Push, SW5 SW_Push, SW6 SW_Push, SW7 SW_Push, SW8 SW_Push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

Commit message: Add files via upload
Connections:
- J1 pad 1: SCL -> GND
- J1 pad 2: SDA -> +3V3
- J1 pad 3: +3V3 -> SDA
- J1 pad 4: GND -> SCL
Routing:
- net GND: track 84.1 -> 92.4 mm
- net SCL: track 29.6 -> 23.1 mm
- net +3V3: track 45.6 -> 44.6 mm
- net SDA: track 24.2 -> 23.1 mm
Changed lines of the file:
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@@
 			(drillshape 0)
 			(scaleselection 1)
-			(outputdirectory "../../")
+			(outputdirectory "C:/Users/loren/Desktop/")
 		)
 	)
@@
 			(layers "*.Cu" "*.Mask")
 			(remove_unused_layers no)
-			(net 19 "SCL")
+			(net 13 "GND")
 			(pinfunction "Pin_1")
 			(pintype "passive")
@@
 			(layers "*.Cu" "*.Mask")
 			(remove_unused_layers no)
-			(net 18 "SDA")
+			(net 17 "+3V3")
 			(pinfunction "Pin_2")
 			(pintype "passive")
@@
 			(layers "*.Cu" "*.Mask")
 			(remove_unused_layers no)
-			(net 17 "+3V3")
+			(net 18 "SDA")
 			(pinfunction "Pin_3")
 			(pintype "passive")
@@
 			(layers "*.Cu" "*.Mask")
 			(remove_unused_layers no)
-			(net 13 "GND")
+			(net 19 "SCL")
 			(pinfunction "Pin_4")
 			(pintype "passive")
@@
 	)
 	(segment
+		(start 130.6955 67.044)
+		(end 129.8955 67.044)
+		(width 0.2)
+		(layer "B.Cu")
+		(net 13)
+	)
+	(segment
 		(start 117.991 60.968)
 		(end 106.68 49.657)
@@
 	)
 	(segment
+		(start 140.1825 67.044)
+		(end 140.272414 67.044)
+		(width 0.2)
+		(layer "B.Cu")
+		(net 13)
+	)
+	(segment
 		(start 88.118 51.825)
 		(end 103.42424 51.825)
@@
 	)
 	(segment
-		(start 141.2835 66.032914)
-		(end 141.2835 62.8235)
+		(start 146.185 53.336)
+		(end 146.185 61.689825)
 		(width 0.2)
 		(layer "B.Cu")
@@
 	)
 	(segment
-		(start 141.2835 62.8235)
-		(end 141.732 62.375)
+		(start 141.2835 66.032914)
+		(end 141.2835 64.6434)
 		(width 0.2)
 		(layer "B.Cu")
@@
 	)
 	(segment
-		(start 141.732 62.375)
-		(end 141.732 59.805)
+		(start 134.1325 63.607)
+		(end 130.6955 67.044)
 		(width 0.2)
 		(layer "B.Cu")
@@
 	)
 	(segment
-		(start 129.8955 67.044)
-		(end 131.026 67.044)
+		(start 140.2471 63.607)
+		(end 134.1325 63.607)
 		(width 0.2)
 		(layer "B.Cu")
@@
 	)
 	(segment
-		(start 130.9965 66.032914)
-		(end 130.9965 65.055086)
+		(start 145.034 52.185)
+		(end 146.185 53.336)
 		(width 0.2)
 		(layer "B.Cu")
@@
 	)
 	(segment
-		(start 145.034 59.805)
-		(end 141.732 59.805)
+		(start 140.830825 67.044)
+		(end 140.1825 67.044)
 		(width 0.2)
 		(layer "B.Cu")
@@
 	)
 	(segment
-		(start 138.265 59.805)
-		(end 141.732 59.805)
+		(start 130.9965 66.032914)
+		(end 130.9965 65.055086)
 		(width 0.2)
 		(layer "B.Cu")
@@
 	)
 	(segment
-		(start 140.1825 67.044)
-		(end 140.272414 67.044)
+		(start 141.2835 64.6434)
+		(end 140.2471 63.607)
 		(width 0.2)
 		(layer "B.Cu")
@@
 	)
 	(segment
-		(start 131.026 67.044)
-		(end 138.265 59.805)
+		(start 146.185 61.689825)
+		(end 140.830825 67.044)
 		(width 0.2)
 		(layer "B.Cu")
@@
 	)
 	(segment
-		(start 126.966 45.966)
-		(end 138.265 57.265)
-		(width 0.2)
-		(layer "F.Cu")
-		(net 17)
-	)
-	(segment
-		(start 138.265 57.265)
-		(end 145.034 57.265)
+		(start 112.911 45.966)
+		(end 106.68 52.197)
 		(width 0.2)
 		(layer "F.Cu")
@@
 	)
 	(segment
-		(start 106.68 52.197)
+		(start 136.275 45.966)
 		(end 112.911 45.966)
 		(width 0.2)
@@
 	)
 	(segment
-		(start 112.911 45.966)
-		(end 126.966 45.966)
+		(start 145.034 54.725)
+		(end 136.275 45.966)
 		(width 0.2)
 		(layer "F.Cu")
@@
 	)
 	(segment
-		(start 121.93 57.277)
-		(end 139.18 57.277)
-		(width 0.2)
-		(layer "B.Cu")
-		(net 18)
-	)
-	(segment
-		(start 141.732 54.725)
-		(end 145.034 54.725)
+		(start 121.942 57.265)
+		(end 121.93 57.277)
 		(width 0.2)
 		(layer "B.Cu")
@@
 	)
 	(segment
-		(start 139.18 57.277)
-		(end 141.732 54.725)
+		(start 145.034 57.265)
+		(end 121.942 57.265)
 		(width 0.2)
 		(layer "B.Cu")
@@
 	)
 	(segment
-		(start 121.93 59.817)
-		(end 120.829 58.716)
-		(width 0.2)
-		(layer "B.Cu")
-		(net 19)
-	)
-	(segment
-		(start 120.829 56.80024)
-		(end 121.74124 55.888)
+		(start 121.942 59.805)
+		(end 121.93 59.817)
 		(width 0.2)
 		(layer "B.Cu")
@@
 	)
 	(segment
-		(start 141.732 52.185)
-		(end 145.034 52.185)
-		(width 0.2)
-		(layer "B.Cu")
-		(net 19)
-	)
-	(segment
-		(start 121.74124 55.888)
-		(end 138.029 55.888)
-		(width 0.2)
-		(layer "B.Cu")
-		(net 19)
-	)
-	(segment
-		(start 120.829 58.716)
-		(end 120.829 56.80024)
-		(width 0.2)
-		(layer "B.Cu")
-		(net 19)
-	)
-	(segment
-		(start 138.029 55.888)
-		(end 141.732 52.185)
+		(start 145.034 59.805)
+		(end 121.942 59.805)
 		(width 0.2)
 		(layer "B.Cu")
